File: Projects/mbed 6LoWPAN Border Router HAT/mbed 6LoWPAN Border Router HAT.brd (EAGLE design)
At the start: 65 x 56.5 mm, 84 parts, among them CON1 TC2030-CTX-NL, CON2 USB_MICROB, IC1 CAT24C32WI-GT3, IC2 74LVC1G08SE-7, IC3 MK64FN1M0VLL12, IC4 LPC11U35FHI33/501, IC5 USBLC6-2SC6, IC6 LD1117S33, Q1 32.768kHz, Q2 12MHz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

Commit message: Updated sch and brd for final build
Parts:
- added RESET-EN: RESET, mbed-HDK:1X03
- R21: value 470R -> 220R
- moved JP1 5.90 mm to (50.6, -18.6)
- moved TP2 3.66 mm to (50.6, -24.0)
- moved TP1 3.36 mm to (50.6, -26.2)
- moved TP16 0.41 mm to (50.6, -4.72)
Connections:
- new net NC: RESET-EN.3
- net GND: now also RESET-EN.2
- net RPI_K64F_RESET: now also RESET-EN.1
Routing:
- net K64F_DAPLINK_TX: track 81.1 -> 75.6 mm
- net RPI_K64F_RESET: track 77.4 -> 82.7 mm
- net K64F_DAPLINK_RX: track 81.8 -> 77.2 mm
Other:
- board text added: "Off"
- board text added: "On"
