File: Projects/mbed 6LoWPAN Border Router HAT/mbed 6LoWPAN Border Router HAT.brd (EAGLE design)
At the start: 65 x 56.5 mm, 85 parts, among them CON1 TC2030-CTX-NL, CON2 USB_MICROB, IC1 CAT24C32WI-GT3, IC2 74LVC1G08SE-7, IC3 MK64FN1M0VLL12, IC4 LPC11U35FHI33/501, IC5 USBLC6-2SC6, IC6 LD1117S33, Q1 32.768kHz, Q2 12MHz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

Commit message: Added all output CAM files V_1_1
Parts:
- JP1: value DEBUG -> 1X03
- RESET-EN: value RESET -> 1X03
Connections:
- removed net NC: RESET-EN.3
Changed lines of the file:
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@@
 <attribute name="VALUE" x="30.607" y="-46.736" size="1.27" layer="27" rot="R90"/>
 </element>
-<element name="JP1" library="mbed-HDK" package="1X03" value="DEBUG" x="50.5968" y="-18.5928" locked="yes" smashed="yes" rot="R90">
+<element name="JP1" library="mbed-HDK" package="1X03" value="1X03" x="50.5968" y="-18.5928" locked="yes" smashed="yes" rot="R90">
 <attribute name="NAME" x="48.768" y="-19.5072" size="0.8128" layer="25" font="vector" ratio="12" rot="R90"/>
 <attribute name="VALUE" x="53.7718" y="-22.4028" size="1.27" layer="27" rot="R90"/>
@@
 <attribute name="VALUE" x="-1.016" y="-26.289" size="1.016" layer="27" font="vector" ratio="12" rot="R90"/>
 </element>
-<element name="RESET-EN" library="mbed-HDK" package="1X03" value="RESET" x="50.5968" y="-10.2108" locked="yes" smashed="yes" rot="R270">
+<element name="RESET-EN" library="mbed-HDK" package="1X03" value="1X03" x="50.5968" y="-10.2108" locked="yes" smashed="yes" rot="R270">
 <attribute name="NAME" x="48.768" y="-13.1064" size="0.8128" layer="25" font="vector" ratio="12" rot="R90"/>
 <attribute name="VALUE" x="46.7868" y="-6.4008" size="1.016" layer="27" font="vector" ratio="12" rot="R270"/>
@@
 <wire x1="36.068" y1="-45.032" x2="36.1062" y2="-44.9938" width="0.1524" layer="1"/>
 </signal>
-<signal name="NC">
-<contactref element="RESET-EN" pad="3"/>
-</signal>
 </signals>

Commit message: Final version V_1_1 of Border Router Hat Job
Routing:
- net +3.3V: track 19.8 -> 2.03 mm, vias 3 -> 0
Changed lines of the file:
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@@
 <attribute name="VALUE" x="38.517" y="-31.802" size="1.27" layer="27" rot="R270"/>
 </element>
-<element name="R8" library="mbed-HDK" package="0402" value="10k" x="48.5394" y="-47.1932" smashed="yes" rot="R270">
+<element name="R8" library="mbed-HDK" package="0402" value="10k" x="48.5394" y="-47.1932" locked="yes" smashed="yes" rot="R270">
 <attribute name="NAME" x="49.5554" y="-49.4792" size="0.8128" layer="25" font="vector" ratio="12" rot="R90"/>
 <attribute name="VALUE" x="46.6344" y="-46.5582" size="1.27" layer="27" rot="R270"/>
 </element>
-<element name="C4" library="mbed-HDK" package="0402" value="100nF" x="47.1424" y="-47.1678" smashed="yes" rot="R270">
+<element name="C4" library="mbed-HDK" package="0402" value="100nF" x="47.1424" y="-47.1678" locked="yes" smashed="yes" rot="R270">
 <attribute name="NAME" x="48.4124" y="-49.4538" size="0.8128" layer="25" font="vector" ratio="12" rot="R90"/>
 <attribute name="VALUE" x="45.2374" y="-46.5328" size="1.27" layer="27" rot="R270"/>
@@
 <attribute name="NAME" x="-3.81" y="-21.209" size="0.8128" layer="21" font="vector" ratio="12"/>
 </element>
-<element name="R15" library="mbed-HDK" package="0402" value="10k" x="51.816" y="-41.021" smashed="yes" rot="R270">
+<element name="R15" library="mbed-HDK" package="0402" value="10k" x="51.816" y="-41.021" locked="yes" smashed="yes" rot="R270">
 <attribute name="NAME" x="52.578" y="-43.9928" size="0.8128" layer="21" font="vector" ratio="12" rot="R90"/>
 </element>
-<element name="IC2" library="mbed-HDK" package="SOT353" value="74LVC1G08SE-7" x="36.9062" y="-45.6438" smashed="yes" rot="R90">
+<element name="IC2" library="mbed-HDK" package="SOT353" value="74LVC1G08SE-7" x="36.9062" y="-45.6438" locked="yes" smashed="yes" rot="R90">
 <attribute name="NAME" x="35.9722" y="-44.6232" size="0.8128" layer="25" font="vector" ratio="12"/>
 <attribute name="VALUE" x="39.5062" y="-47.5938" size="1.016" layer="27" font="vector" ratio="12" rot="R90"/>
 </element>
-<element name="R6" library="mbed-HDK" package="0402" value="10k" x="36.449" y="-47.752" smashed="yes">
+<element name="R6" library="mbed-HDK" package="0402" value="10k" x="36.449" y="-47.752" locked="yes" smashed="yes">
 <attribute name="NAME" x="35.814" y="-49.149" size="0.8128" layer="25" font="vector" ratio="12"/>
 <attribute name="VALUE" x="35.179" y="-51.562" size="1.016" layer="27" font="vector" ratio="12"/>
 </element>
-<element name="R9" library="mbed-HDK" package="0402" value="1k" x="34.671" y="-45.974" smashed="yes" rot="R90">
+<element name="R9" library="mbed-HDK" package="0402" value="1k" x="34.671" y="-45.974" locked="yes" smashed="yes" rot="R90">
 <attribute name="NAME" x="32.766" y="-48.26" size="0.8128" layer="25" font="vector" ratio="12"/>
 <attribute name="VALUE" x="38.481" y="-47.244" size="1.016" layer="27" font="vector" ratio="12" rot="R90"/>
@@
 <wire x1="35.767" y1="-27.302" x2="35.7632" y2="-27.2982" width="0.1524" layer="1"/>
 <wire x1="35.7632" y1="-27.2982" x2="35.7632" y2="-25.273" width="0.1524" layer="1"/>
-<via x="23.368" y="-7.62" extent="1-16" drill="0.254"/>
-<via x="35.941" y="-8.509" extent="1-16" drill="0.254"/>
-<via x="40.894" y="-8.509" extent="1-16" drill="0.254"/>
-<wire x1="35.941" y1="-8.509" x2="40.767" y2="-8.509" width="0.6096" layer="16"/>
-<wire x1="23.368" y1="-7.62" x2="24.257" y2="-8.509" width="0.6096" layer="16"/>
-<wire x1="24.257" y1="-8.509" x2="35.941" y2="-8.509" width="0.6096" layer="16"/>
 <contactref element="IC2" pad="5"/>
 <contactref element="R6" pad="1"/>
@@
 <wire x1="45.847" y1="-10.795" x2="44.45" y2="-9.398" width="0.1524" layer="16"/>
 <wire x1="44.45" y1="-9.398" x2="21.844" y2="-9.398" width="0.1524" layer="16"/>
-<wire x1="21.844" y1="-9.398" x2="14.097" y2="-1.651" width="0.1524" layer="16"/>
 <via x="14.097" y="-1.651" extent="1-16" drill="0.254"/>
 <wire x1="14.097" y1="-1.651" x2="9.144" y2="-1.651" width="0.1524" layer="1"/>
@@
 <wire x1="8.89" y1="-1.397" x2="8.89" y2="1.27" width="0.1524" layer="1"/>
 <wire x1="8.89" y1="1.27" x2="7.62" y2="2.54" width="0.1524" layer="1"/>
+<wire x1="21.844" y1="-9.398" x2="14.097" y2="-1.651" width="0.1524" layer="16"/>
 </signal>
 <signal name="K64F_RPI_CTS">
