File: Projects/mbed 6LoWPAN Border Router HAT/mbed 6LoWPAN Border Router HAT.sch (EAGLE design)
At the start: 83 parts, among them CON1 TC2030-CTX-NL, CON2 USB_MICROB, IC1 CAT24C32WI-GT3, IC2 74LVC1GXX, IC3 MK64FN1M0VLL12, IC4 LPC11U35FHI33/501, IC5 USBLC6-2SC6, IC6 LD1117S33, Q1 32.768kHz, Q2 12MHz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

Commit message: Updated 6LoWPAN Border Router HDK to Rev 1.1
Parts:
- added D3: BAT60J, mbed-HDK:BAT60A
- R9: value 10k -> 1k
Connections:
- net N$5: now also D3.K
- net TGT_NRESET: now also D3.A
Changed lines of the file:
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@@
 <?xml version="1.0" encoding="utf-8"?>
 <!DOCTYPE eagle SYSTEM "eagle.dtd">
-<eagle version="7.3.0">
+<eagle version="7.6.0">
 <drawing>
 <settings>
@@
 <part name="R6" library="mbed-HDK" deviceset="R" device="0402" value="10k"/>
 <part name="PWR6" library="mbed-HDK" deviceset="+3.3V" device=""/>
-<part name="R9" library="mbed-HDK" deviceset="R" device="0402" value="10k"/>
+<part name="R9" library="mbed-HDK" deviceset="R" device="0402" value="1k"/>
+<part name="D3" library="mbed-HDK" deviceset="BAT60A" device="" value="BAT60J"/>
 </parts>
 <sheets>
@@
 </instance>
 <instance part="GND30" gate="1" x="190.5" y="66.04" smashed="yes" rot="R90"/>
+<instance part="D3" gate="G$1" x="93.98" y="160.02"/>
 </instances>
 <busses>
@@
 <wire x1="109.22" y1="160.02" x2="109.22" y2="152.4" width="0.1524" layer="91"/>
 <junction x="109.22" y="160.02"/>
+<pinref part="D3" gate="G$1" pin="K"/>
+<wire x1="96.52" y1="160.02" x2="109.22" y2="160.02" width="0.1524" layer="91"/>
 </segment>
 </net>
@@
 </segment>
 </net>
+<net name="TGT_NRESET" class="0">
+<segment>
+<pinref part="D3" gate="G$1" pin="A"/>
+<wire x1="91.44" y1="160.02" x2="86.36" y2="160.02" width="0.1524" layer="91"/>
+<label x="76.2" y="162.56" size="1.778" layer="95" font="vector" ratio="12"/>
+</segment>
+</net>

Commit message: Cleaned Schematic
Other:
- note added: "R14 denotes it is NOT FRDM-K64F R15 denotes it is NOT USB SLIP"
- note removed: "R12 denotes it is NOT FRDM-K64F R13 denotes it is NOT USB SLIP"
Changed lines of the file:
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@@
 <plain>
 <text x="43.18" y="93.98" size="1.778" layer="97" font="vector" ratio="12">TGT_SWCLK is also EZP_CK</text>
-<text x="228.6" y="154.94" size="1.6764" layer="97" font="vector" ratio="12">R12 denotes it is NOT FRDM-K64F
-R13 denotes it is NOT USB SLIP</text>
+<text x="228.6" y="154.94" size="1.6764" layer="97" font="vector" ratio="12">R14 denotes it is NOT FRDM-K64F
+R15 denotes it is NOT USB SLIP</text>
 </plain>
 <instances>

Commit message: Cleaned up silk screen
Parts:
- IC2: value 74LVC1GXX -> 74LVC1G08SE-7
Changed lines of the file:
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@@
 <part name="R15" library="mbed-HDK" deviceset="R" device="0402" value="10k"/>
 <part name="GND21" library="mbed-HDK" deviceset="GND" device=""/>
-<part name="IC2" library="mbed-HDK" deviceset="74LVC1GXX" device=""/>
+<part name="IC2" library="mbed-HDK" deviceset="74LVC1GXX" device="" value="74LVC1G08SE-7"/>
 <part name="PWR9" library="mbed-HDK" deviceset="+3.3V" device=""/>
 <part name="GND10" library="mbed-HDK" deviceset="GND" device=""/>

Commit message: Updated sch and brd for final build
Parts:
- added RESET-EN: RESET, mbed-HDK:PINHD-1X3
- R21: value 470R -> 220R
Connections:
- new net NC: RESET-EN.3
- net GND: now also RESET-EN.2
- net RPI_K64F_RESET: now also RESET-EN.1
Other:
- moved on the sheet: C10, C11, C12, C13, C6, C7, C8, C9, CON1, JP1

Commit message: Added all output CAM files V_1_1
Parts:
- JP1: value DEBUG -> 1X03
- RESET-EN: value RESET -> 1X03
Connections:
- removed net NC: RESET-EN.3
Changed lines of the file:
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@@
 <part name="PWR10" library="mbed-HDK" deviceset="+3.3V" device=""/>
 <part name="GND13" library="mbed-HDK" deviceset="GND" device=""/>
-<part name="JP1" library="mbed-HDK" deviceset="PINHD-1X3" device="" value="DEBUG"/>
+<part name="JP1" library="mbed-HDK" deviceset="PINHD-1X3" device="" value="1X03"/>
 <part name="GND18" library="mbed-HDK" deviceset="GND" device=""/>
 <part name="R20" library="mbed-HDK" deviceset="R" device="0402" value="10k"/>
@@
 <part name="R9" library="mbed-HDK" deviceset="R" device="0402" value="1k"/>
 <part name="D3" library="mbed-HDK" deviceset="BAT60A" device="" value="BAT60J"/>
-<part name="RESET-EN" library="mbed-HDK" deviceset="PINHD-1X3" device="" value="RESET"/>
+<part name="RESET-EN" library="mbed-HDK" deviceset="PINHD-1X3" device="" value="1X03"/>
 <part name="GND36" library="mbed-HDK" deviceset="GND" device=""/>
 </parts>
@@
 </segment>
 </net>
-<net name="NC" class="0">
-<segment>
-<pinref part="RESET-EN" gate="A" pin="3"/>
-<wire x1="142.24" y1="12.7" x2="154.94" y2="12.7" width="0.1524" layer="91"/>
-<label x="154.94" y="12.7" size="1.778" layer="95" font="vector" ratio="12"/>
-</segment>
-</net>
