File: Production Design Projects/mbed 6LoWPAN Border Router HAT/v1.1.0/mbed 6LoWPAN Border Router HAT.brd (EAGLE design)
At the start: 65 x 56.5 mm, 85 parts, among them CON1 TC2030-CTX-NL, CON2 USB_MICROB, IC1 CAT24C32WI-GT3, IC2 74LVC1G08SE-7, IC3 MK64FN1M0VLL12, IC4 LPC11U35FHI33/501, IC5 USBLC6-2SC6, IC6 LD1117S33, Q1 32.768kHz, Q2 12MHz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

Commit message: Updated Readme
Parts:
- removed D3: BAT60J, mbed-HDK:BAT60A
- added D4: BAT60J, mbed-HDK:SOD323
- D1, D2: device mbed-HDK:BAT60A -> mbed-HDK:SOD323
Connections:
- net N$5: now also D4.K; no longer D3.K
- net TGT_NRESET: now also D4.A; no longer D3.A
