File: Production Design Projects/mbed 6LoWPAN Border Router HAT/v1.1.0/mbed 6LoWPAN Border Router HAT.sch (EAGLE design)
At the start: 85 parts, among them CON1 TC2030-CTX-NL, CON2 USB_MICROB, IC1 CAT24C32WI-GT3, IC2 74LVC1G08SE-7, IC3 MK64FN1M0VLL12, IC4 LPC11U35FHI33/501, IC5 USBLC6-2SC6, IC6 LD1117S33, Q1 32.768kHz, Q2 12MHz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

Commit message: Updated Readme
Parts:
- removed D3: BAT60J, mbed-HDK:BAT60A
- added D4: BAT60J, mbed-HDK:BAT60J
Connections:
- net N$5: now also D4.K; no longer D3.K
- net TGT_NRESET: now also D4.A; no longer D3.A
Changed lines of the file:
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@@
 <part name="CON1" library="mbed-HDK" deviceset="TC2030-CTX" device="-NL"/>
 <part name="PWR24" library="mbed-HDK" deviceset="+3.3V" device=""/>
-<part name="D2" library="mbed-HDK" deviceset="BAT60A" device=""/>
+<part name="D2" library="mbed-HDK" deviceset="BAT60A" device="" value="BAT60A"/>
 <part name="PWR5" library="mbed-HDK" deviceset="+3.3V" device=""/>
-<part name="D1" library="mbed-HDK" deviceset="BAT60A" device=""/>
+<part name="D1" library="mbed-HDK" deviceset="BAT60A" device="" value="BAT60A"/>
 <part name="TP2" library="mbed-HDK" deviceset="TEST-POINT" device="-50R-PTH" value="TEST-POINT-50R-PTH"/>
 <part name="GND1" library="mbed-HDK" deviceset="GND" device=""/>
@@
 <part name="PWR6" library="mbed-HDK" deviceset="+3.3V" device=""/>
 <part name="R9" library="mbed-HDK" deviceset="R" device="0402" value="1k"/>
-<part name="D3" library="mbed-HDK" deviceset="BAT60A" device="" value="BAT60J"/>
 <part name="RESET-EN" library="mbed-HDK" deviceset="PINHD-1X3" device="" value="1X03"/>
 <part name="GND36" library="mbed-HDK" deviceset="GND" device=""/>
+<part name="D4" library="mbed-HDK" deviceset="BAT60J" device=""/>
 </parts>
 <sheets>
@@
 </instance>
 <instance part="GND30" gate="1" x="190.5" y="66.04" smashed="yes" rot="R90"/>
-<instance part="D3" gate="G$1" x="93.98" y="160.02"/>
+<instance part="D4" gate="G$1" x="93.98" y="160.02"/>
 </instances>
 <busses>
@@
 <wire x1="109.22" y1="160.02" x2="109.22" y2="152.4" width="0.1524" layer="91"/>
 <junction x="109.22" y="160.02"/>
-<pinref part="D3" gate="G$1" pin="K"/>
 <wire x1="96.52" y1="160.02" x2="109.22" y2="160.02" width="0.1524" layer="91"/>
+<pinref part="D4" gate="G$1" pin="K"/>
 </segment>
 </net>
@@
 <net name="TGT_NRESET" class="0">
 <segment>
-<pinref part="D3" gate="G$1" pin="A"/>
 <wire x1="91.44" y1="160.02" x2="86.36" y2="160.02" width="0.1524" layer="91"/>
 <label x="76.2" y="162.56" size="1.778" layer="95" font="vector" ratio="12"/>
-</segment>
-</net>
+<pinref part="D4" gate="G$1" pin="A"/>
+</segment>
+</net>
