File: Production Design Projects/mbedXdotShield/v1.0.0/MBEDxDOT.sch (EAGLE design)
At the start: 68 parts, among them CON1 47346-0001, CON2 S2B-PH-SM4-TB(LF)(SN), Q1 12MHz, SW2 SKRKAEE010, T1 BSS84, U1 MTXDOT-EU1-A00-1, U2 TLV73333PDBVT, U3 AT45DB321E-SHF-B

Commit message: Final release of V1.0.0
Parts:
- added R27: 0, mbed-HDK-RLCQ:RESISTOR0402
- added SW3: JS202011JCQN, mbed-HDK-Switch:JS202011JCQN
- renumbered SW2 to GPIO1
Connections:
- new net N$49: BRD1.3V3, BRD1.IOREF, R27.P$1
- new net N$50: R17.P$2, SW3.6
- new net N$51: R18.P$2, SW3.2
- net +3.3V_TGT: now also R27.P$2; no longer BRD1.3V3, BRD1.IOREF
- net UART1_RX: now also SW3.3, SW3.5; no longer R17.P$2
- net UART1_TX: now also SW3.1, SW3.7; no longer R18.P$2
Other:
- note added: "UART Swap - DPDT Switch"
Changed lines of the file:
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@@
 <part name="PWR5" library="mbed-HDK-misc-Symbol" deviceset="+3.3V_TGT" device=""/>
 <part name="GND24" library="mbed-HDK-misc-Symbol" deviceset="GND" device=""/>
-<part name="SW2" library="mbed-HDK-Switch" deviceset="SKRKAEE010" device=""/>
+<part name="GPIO1" library="mbed-HDK-Switch" deviceset="SKRKAEE010" device=""/>
 <part name="GND25" library="mbed-HDK-misc-Symbol" deviceset="GND" device=""/>
 <part name="PWR7" library="mbed-HDK-misc-Symbol" deviceset="+3.3V_TGT" device=""/>
@@
 <part name="C16" library="mbed-HDK-RLCQ" deviceset="CAPACITOR" device="0603" value="10uF"/>
 <part name="GND32" library="mbed-HDK-misc-Symbol" deviceset="GND" device=""/>
+<part name="R27" library="mbed-HDK-RLCQ" deviceset="RESISTOR" device="0402" value="0"/>
+<part name="SW3" library="mbed-HDK-Switch" deviceset="JS202011JCQN" device=""/>
 </parts>
 <sheets>
@@
 </instance>
 <instance part="GND24" gate="1" x="137.16" y="83.82" rot="R90"/>
-<instance part="SW2" gate="G$1" x="129.54" y="83.82"/>
+<instance part="GPIO1" gate="G$1" x="129.54" y="83.82"/>
 <instance part="LED1" gate="G$1" x="61.468" y="83.058"/>
 <instance part="GND19" gate="1" x="61.468" y="70.358"/>
@@
 <wire x1="134.62" y1="83.82" x2="137.16" y2="83.82" width="0.1524" layer="91"/>
 <pinref part="GND24" gate="1" pin="GND"/>
-<pinref part="SW2" gate="G$1" pin="S"/>
+<pinref part="GPIO1" gate="G$1" pin="S"/>
 </segment>
 <segment>
@@
 <label x="109.22" y="83.82" size="2.286" layer="90"/>
 <junction x="119.38" y="83.82"/>
-<pinref part="SW2" gate="G$1" pin="P"/>
+<pinref part="GPIO1" gate="G$1" pin="P"/>
 </segment>
 </net>
@@
 <text x="123.698" y="139.446" size="2.54" layer="91">Board Headers</text>
 <text x="2.54" y="180.34" size="6.4516" layer="90">BOARD HEADERS</text>
+<text x="184.658" y="60.706" size="2.54" layer="91">UART Swap - DPDT Switch</text>
 </plain>
 <instances>
@@
 <instance part="GND22" gate="1" x="104.14" y="101.6" rot="R270"/>
 <instance part="GND25" gate="1" x="162.56" y="119.38" rot="R90"/>
-<instance part="PWR7" gate="G$1" x="78.74" y="119.38" smashed="yes">
-<attribute name="VALUE" x="79.248" y="124.206" size="2.286" layer="92" rot="R90"/>
+<instance part="PWR7" gate="G$1" x="78.74" y="129.54" smashed="yes">
+<attribute name="VALUE" x="79.248" y="134.366" size="2.286" layer="92" rot="R90"/>
 </instance>
 <instance part="BRD1" gate="G$1" x="111.76" y="134.62"/>
@@
 <attribute name="VALUE" x="170.434" y="128.016" size="1.27" layer="96" font="vector" ratio="12"/>
 </instance>
+<instance part="R27" gate="G$1" x="78.74" y="121.92" smashed="yes" rot="R90">
+<attribute name="NAME" x="77.724" y="115.824" size="1.27" layer="95" font="vector" ratio="12" rot="R90"/>
+<attribute name="VALUE" x="77.724" y="124.714" size="1.27" layer="96" font="vector" ratio="12" rot="R90"/>
+</instance>
+<instance part="SW3" gate="G$1" x="198.12" y="83.82"/>
 </instances>
 <busses>
@@
 </segment>
 </net>
-<net name="+3.3V_TGT" class="0">
-<segment>
-<pinref part="PWR7" gate="G$1" pin="+3.3V_TGT"/>
-<wire x1="78.74" y1="109.22" x2="78.74" y2="114.3" width="0.1524" layer="91"/>
-<wire x1="78.74" y1="114.3" x2="78.74" y2="119.38" width="0.1524" layer="91"/>
-<wire x1="106.68" y1="109.22" x2="78.74" y2="109.22" width="0.1524" layer="91"/>
-<pinref part="BRD1" gate="G$1" pin="3V3"/>
-<wire x1="106.68" y1="114.3" x2="78.74" y2="114.3" width="0.1524" layer="91"/>
-<junction x="78.74" y="114.3"/>
-<pinref part="BRD1" gate="G$1" pin="IOREF"/>
-</segment>
-</net>
 <net name="SPI_SCK" class="0">
 <segment>
@@
 </segment>
 </net>
-<net name="UART1_TX" class="0">
-<segment>
-<junction x="177.8" y="83.82"/>
-<label x="177.8" y="83.82" size="2.286" layer="90"/>
-<pinref part="R18" gate="G$1" pin="P$2"/>
-<wire x1="172.72" y1="83.82" x2="177.8" y2="83.82" width="0.1524" layer="91"/>
-</segment>
-</net>
-<net name="UART1_RX" class="0">
-<segment>
-<junction x="177.8" y="81.28"/>
-<label x="177.8" y="81.28" size="2.286" layer="90"/>
-<pinref part="R17" gate="G$1" pin="P$2"/>
-<wire x1="172.72" y1="81.28" x2="177.8" y2="81.28" width="0.1524" layer="91"/>
-</segment>
-</net>
 <net name="GPIO3" class="0">
 <segment>
@@
 <pinref part="D1" gate="G$1" pin="A"/>
 <wire x1="63.5" y1="106.68" x2="58.42" y2="106.68" width="0.1524" layer="91"/>
-<wire x1="58.42" y1="106.68" x2="58.42" y2="121.92" width="0.1524" layer="91"/>
-<junction x="58.42" y="121.92"/>
-<label x="58.674" y="122.936" size="2.286" layer="92" rot="R90"/>
+<wire x1="58.42" y1="106.68" x2="58.42" y2="132.08" width="0.1524" layer="91"/>
+<junction x="58.42" y="132.08"/>
+<label x="58.674" y="133.096" size="2.286" layer="92" rot="R90"/>
 </segment>
 </net>
@@
 </segment>
 </net>
+<net name="N$49" class="0">
+<segment>
+<wire x1="78.74" y1="109.22" x2="78.74" y2="114.3" width="0.1524" layer="91"/>
+<wire x1="106.68" y1="109.22" x2="78.74" y2="109.22" width="0.1524" layer="91"/>
+<pinref part="BRD1" gate="G$1" pin="3V3"/>
+<wire x1="106.68" y1="114.3" x2="78.74" y2="114.3" width="0.1524" layer="91"/>
+<pinref part="BRD1" gate="G$1" pin="IOREF"/>
+<pinref part="R27" gate="G$1" pin="P$1"/>
+<wire x1="78.74" y1="114.3" x2="78.74" y2="116.84" width="0.1524" layer="91"/>
+<junction x="78.74" y="114.3"/>
+</segment>
+</net>
+<net name="+3.3V_TGT" class="0">
+<segment>
+<pinref part="R27" gate="G$1" pin="P$2"/>
+<pinref part="PWR7" gate="G$1" pin="+3.3V_TGT"/>
+<wire x1="78.74" y1="127" x2="78.74" y2="129.54" width="0.1524" layer="91"/>
+</segment>
+</net>
+<net name="N$50" class="0">
+<segment>
+<pinref part="R17" gate="G$1" pin="P$2"/>
+<wire x1="172.72" y1="81.28" x2="187.96" y2="81.28" width="0.1524" layer="91"/>
+<wire x1="187.96" y1="81.28" x2="187.96" y2="73.66" width="0.1524" layer="91"/>
+<pinref part="SW3" gate="G$1" pin="6"/>
+<wire x1="187.96" y1="73.66" x2="198.12" y2="73.66" width="0.1524" layer="91"/>
+</segment>
+</net>
+<net name="N$51" class="0">
+<segment>
+<pinref part="R18" gate="G$1" pin="P$2"/>
+<wire x1="172.72" y1="83.82" x2="198.12" y2="83.82" width="0.1524" layer="91"/>
+<pinref part="SW3" gate="G$1" pin="2"/>
+</segment>
+</net>
+<net name="UART1_TX" class="0">
+<segment>
+<pinref part="SW3" gate="G$1" pin="1"/>
+<wire x1="213.36" y1="86.36" x2="220.98" y2="86.36" width="0.1524" layer="91"/>
+<junction x="220.98" y="86.36"/>
+<label x="220.98" y="86.36" size="2.286" layer="90"/>
+</segment>
+<segment>
+<pinref part="SW3" gate="G$1" pin="7"/>
+<wire x1="213.36" y1="71.12" x2="220.98" y2="71.12" width="0.1524" layer="91"/>
+<junction x="220.98" y="71.12"/>
+<label x="220.98" y="71.12" size="2.286" layer="90"/>
+</segment>
+</net>
+<net name="UART1_RX" class="0">
+<segment>
+<pinref part="SW3" gate="G$1" pin="3"/>
+<wire x1="213.36" y1="81.28" x2="220.98" y2="81.28" width="0.1524" layer="91"/>
+<junction x="220.98" y="81.28"/>
+<label x="220.98" y="81.28" size="2.286" layer="90"/>
+</segment>
+<segment>
+<pinref part="SW3" gate="G$1" pin="5"/>
+<wire x1="213.36" y1="76.2" x2="220.98" y2="76.2" width="0.1524" layer="91"/>
+<junction x="220.98" y="76.2"/>
+<label x="220.98" y="76.2" size="2.286" layer="90"/>
+</segment>
+</net>

Commit message: Change part to D6 to BAT60J
Parts:
- D6: value BAT60A -> BAT60J; device mbed-HDK-Transistor:BAT60A -> mbed-HDK-Transistor:BAT60J
Changed lines of the file:
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@@
 <part name="D5" library="mbed-HDK-Transistor" deviceset="BAT60A" device=""/>
 <part name="PWR6" library="mbed-HDK-misc-Symbol" deviceset="+3.3V_TGT" device=""/>
-<part name="D6" library="mbed-HDK-Transistor" deviceset="BAT60A" device=""/>
 <part name="DWG3" library="mbed-HDK-misc-Template" deviceset="MBED-HDK" device=""/>
 <part name="DWG4" library="mbed-HDK-misc-Template" deviceset="MBED-HDK" device=""/>
@@
 <part name="R27" library="mbed-HDK-RLCQ" deviceset="RESISTOR" device="0402" value="0"/>
 <part name="SW3" library="mbed-HDK-Switch" deviceset="JS202011JCQN" device=""/>
+<part name="D6" library="mbed-HDK-Transistor" deviceset="BAT60J" device=""/>
 </parts>
 <sheets>
@@
 <pinref part="RESET" gate="G$1" pin="S"/>
 <junction x="91.44" y="114.3"/>
+<wire x1="91.44" y1="114.3" x2="91.44" y2="124.46" width="0.1524" layer="91"/>
 <pinref part="D6" gate="G$1" pin="K"/>
-<wire x1="91.44" y1="114.3" x2="91.44" y2="124.46" width="0.1524" layer="91"/>
 </segment>
 </net>
@@
 </segment>
 <segment>
-<pinref part="D6" gate="G$1" pin="A"/>
 <wire x1="91.44" y1="129.54" x2="91.44" y2="132.08" width="0.1524" layer="91"/>
 <junction x="91.44" y="132.08"/>
 <label x="91.44" y="132.334" size="2.286" layer="90" rot="R90"/>
-</segment>
-</net>
+<pinref part="D6" gate="G$1" pin="A"/>
+</segment>
+</net>
