File: Bare Design Projects/INTERFACE DAPLink/LPC11u35/INTERFACE_LPC11u35.brd (EAGLE design)
At the start: 28 parts, among them CON1 47346-0001, T1 BSS84, U2 TLV1117LV33DCYR

Commit message: Updated schematic
Parts:
- removed Q1: (no value), mbed-HDK-Oscillator:3.2X.2.5
- added Y1: 7M-12.000MAAJ-T, mbed-HDK-Oscillator:3.2X.2.5
- moved C1 70.7 mm to (-7.16, 9.60)
- moved C10 70.7 mm to (6.43, -6.50)
- moved C11 70.7 mm to (4.72, -1.32)
- moved C12 70.7 mm to (3.47, 1.70)
- moved C13 70.7 mm to (5.57, 1.70)
- moved C14 70.7 mm to (5.99, -9.09)
- moved C15 70.7 mm to (11.4, -7.57)
- moved C2 70.7 mm to (-7.16, 11.3)
- moved C3 70.7 mm to (-3.51, 9.60)
- moved C4 70.7 mm to (-3.51, 11.3)
- moved CON1 70.7 mm to (-13.9, 4.88)
- moved D6 70.7 mm to (9.27, -6.27)
- moved LED3 70.7 mm to (-0.15, 0.00), turned to 90 degrees
- moved LED4 70.7 mm to (-0.15, -2.13)
- moved LED5 70.7 mm to (-0.15, -1.07)
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Connections:
- removed net N$34: LED3.C, R11.1
- new net N$2: LED3.A, R11.1
- net +3.3V: no longer LED3.A
- net GND: now also LED3.C
- net N$37: now also Y1.P$3; no longer Q1.P$3
- net N$40: now also Y1.P$1; no longer Q1.P$1
Routing:
- net +3.3V: track 27.8 -> 26.7 mm
- net N$34: track 0.93 -> 0.00 mm
- net N$2: track 0.00 -> 0.93 mm
Other:
- board text added: "COM"
- board text added: "PWR"
- board text removed: "HID"
- board text removed: "UART"

Commit message: Fixed PDF and name errors
Connections:
- net DAP_NRESET renamed TGT_NRESET
- net DAP_RX renamed TGT_RX
- net DAP_SWCLK renamed TGT_SWCLK
- net DAP_SWDIO renamed TGT_SWDIO
- net DAP_TX renamed TGT_TX
- net DAP_USB_D+ renamed TGT_USB_D+
- net DAP_USB_D- renamed TGT_USB_D-
Changed lines of the file:
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@@
 <wire x1="8.7122" y1="-8.8138" x2="8.7122" y2="-5.6388" width="0.1524" layer="1"/>
 </signal>
-<signal name="DAP_RX">
+<signal name="TGT_RX">
 <contactref element="U1" pad="32"/>
 <wire x1="5.778" y1="-3.4772" x2="4.981" y2="-3.4772" width="0.1524" layer="1"/>
@@
 <wire x1="2.1336" y1="-4.572" x2="1.8288" y2="-4.2672" width="0.1524" layer="16"/>
 </signal>
-<signal name="DAP_USB_D-">
+<signal name="TGT_USB_D-">
 <contactref element="R7" pad="1"/>
 <wire x1="2.4257" y1="2.156459375" x2="2.4257" y2="2.733040625" width="0.1524" layer="1"/>
@@
 <wire x1="-11.028" y1="5.4864" x2="-11.0684" y2="5.5268" width="0.1524" layer="1"/>
 </signal>
-<signal name="DAP_USB_D+">
+<signal name="TGT_USB_D+">
 <contactref element="R4" pad="1"/>
 <wire x1="4.51611875" y1="2.156459375" x2="4.51611875" y2="2.95148125" width="0.1524" layer="1"/>
@@
 <wire x1="-0.6096" y1="4.8768" x2="0.762" y2="3.5052" width="0.1524" layer="1"/>
 </signal>
-<signal name="DAP_SWCLK">
+<signal name="TGT_SWCLK">
 <contactref element="U1" pad="16"/>
 <wire x1="10.478" y1="0.0228" x2="10.8432" y2="0.0228" width="0.1524" layer="1"/>
@@
 <wire x1="16.1544" y1="-4.8768" x2="16.4592" y2="-4.572" width="0.1524" layer="16"/>
 </signal>
-<signal name="DAP_SWDIO">
+<signal name="TGT_SWDIO">
 <contactref element="U1" pad="17"/>
 <wire x1="9.878" y1="0.6228" x2="10.5288" y2="0.6228" width="0.1524" layer="1"/>
@@
 <wire x1="16.002" y1="-3.9624" x2="17.0688" y2="-3.9624" width="0.1524" layer="1"/>
 </signal>
-<signal name="DAP_TX">
+<signal name="TGT_TX">
 <contactref element="U1" pad="31"/>
 <wire x1="5.778" y1="-2.9772" x2="4.6682" y2="-2.9772" width="0.1524" layer="1"/>
@@
 <wire x1="-5.334" y1="5.6388" x2="-5.334" y2="3.9624" width="0" layer="19" extent="16-16"/>
 </signal>
-<signal name="DAP_NRESET">
+<signal name="TGT_NRESET">
 <contactref element="U1" pad="8"/>
 <contactref element="D6" pad="A"/>
