File: Bare Design Projects/INTERFACE DAPLink/LPC11u35/INTERFACE_LPC11u35.sch (EAGLE design)
At the start: 28 parts, among them CON1 47346-0001, T1 BSS84, U2 TLV1117LV33DCYR

Commit message: Updated schematic
Parts:
- Y1: value (none) -> 7M-12.000MAAJ-T
- renumbered Q1 to Y1
Connections:
- removed net N$34: LED3.C, R11.P$1
- new net N$2: LED3.A, R11.P$1
- net +3.3V: no longer LED3.A
- net GND: now also LED3.C
Other:
- moved on the sheet: LED3
Changed lines of the file:
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@@
 <part name="PWR5" library="mbed-HDK-misc-Symbol" deviceset="+3.3V" device=""/>
 <part name="U1" library="mbed-HDK-MF-NXP" deviceset="IF_LPC11U35FHI33/501" device=""/>
-<part name="Q1" library="mbed-HDK-Oscillator" deviceset="7M-12.000MAAJ-T" device=""/>
+<part name="Y1" library="mbed-HDK-Oscillator" deviceset="7M-12.000MAAJ-T" device=""/>
 <part name="CON1" library="mbed-HDK-Connector" deviceset="47346-0001" device=""/>
 <part name="U2" library="mbed-HDK-Power" deviceset="TLV1117LV33DCYR" device=""/>
@@
 <part name="GND6" library="mbed-HDK" deviceset="GND" device=""/>
 <part name="PWR6" library="mbed-HDK-misc-Symbol" deviceset="+3.3V" device=""/>
+<part name="GND7" library="mbed-HDK" deviceset="GND" device=""/>
 </parts>
 <sheets>
@@
 <attribute name="VALUE" x="100.076" y="152.146" size="1.27" layer="96" font="vector" ratio="12" rot="R270"/>
 </instance>
-<instance part="LED3" gate="G$1" x="205.74" y="127" rot="R270"/>
+<instance part="LED3" gate="G$1" x="203.2" y="127" rot="R90"/>
 <instance part="LED4" gate="G$1" x="205.74" y="114.3" rot="R270"/>
 <instance part="LED5" gate="G$1" x="205.74" y="101.6" rot="R270"/>
@@
 </instance>
 <instance part="U1" gate="G$1" x="139.7" y="111.76"/>
-<instance part="Q1" gate="G$1" x="104.14" y="55.88"/>
+<instance part="Y1" gate="G$1" x="104.14" y="55.88"/>
 <instance part="CON1" gate="A" x="142.24" y="170.18" rot="R180"/>
 <instance part="U2" gate="G$1" x="195.58" y="162.56"/>
@@
 <attribute name="VALUE" x="237.744" y="180.086" size="2.286" layer="92"/>
 </instance>
+<instance part="GND7" gate="1" x="210.82" y="127" rot="R90"/>
 </instances>
 <busses>
@@
 <pinref part="GND6" gate="1" pin="GND"/>
 </segment>
+<segment>
+<pinref part="LED3" gate="G$1" pin="C"/>
+<wire x1="208.28" y1="127" x2="210.82" y2="127" width="0.1524" layer="91"/>
+<pinref part="GND7" gate="1" pin="GND"/>
+</segment>
 </net>
 <net name="IF_NRESET" class="0">
@@
 </segment>
 </net>
-<net name="N$34" class="0">
-<segment>
-<wire x1="200.66" y1="127" x2="193.04" y2="127" width="0.1524" layer="91"/>
-<pinref part="R11" gate="G$1" pin="P$1"/>
-<pinref part="LED3" gate="G$1" pin="C"/>
-</segment>
-</net>
 <net name="N$35" class="0">
 <segment>
@@
 <pinref part="C15" gate="G$1" pin="P$1"/>
 <pinref part="U1" gate="G$1" pin="XTALOUT"/>
-<pinref part="Q1" gate="G$1" pin="2"/>
+<pinref part="Y1" gate="G$1" pin="2"/>
 </segment>
 </net>
@@
 <pinref part="C14" gate="G$1" pin="P$1"/>
 <pinref part="U1" gate="G$1" pin="XTALIN"/>
-<pinref part="Q1" gate="G$1" pin="1"/>
+<pinref part="Y1" gate="G$1" pin="1"/>
 </segment>
 </net>
@@
 <segment>
 <wire x1="215.9" y1="101.6" x2="215.9" y2="114.3" width="0.1524" layer="91"/>
-<wire x1="215.9" y1="114.3" x2="215.9" y2="127" width="0.1524" layer="91"/>
-<wire x1="215.9" y1="127" x2="215.9" y2="134.62" width="0.1524" layer="91"/>
+<wire x1="215.9" y1="114.3" x2="215.9" y2="134.62" width="0.1524" layer="91"/>
 <wire x1="208.28" y1="101.6" x2="215.9" y2="101.6" width="0.1524" layer="91"/>
 <wire x1="208.28" y1="114.3" x2="215.9" y2="114.3" width="0.1524" layer="91"/>
-<wire x1="208.28" y1="127" x2="215.9" y2="127" width="0.1524" layer="91"/>
-<junction x="215.9" y="127"/>
 <junction x="215.9" y="114.3"/>
-<pinref part="LED3" gate="G$1" pin="A"/>
 <pinref part="LED4" gate="G$1" pin="A"/>
 <pinref part="LED5" gate="G$1" pin="A"/>
@@
 </segment>
 </net>
+<net name="N$2" class="0">
+<segment>
+<pinref part="R11" gate="G$1" pin="P$1"/>
+<pinref part="LED3" gate="G$1" pin="A"/>
+<wire x1="193.04" y1="127" x2="200.66" y2="127" width="0.1524" layer="91"/>
+</segment>
+</net>

Commit message: Fixed PDF and name errors
Connections:
- net DAP_NRESET renamed TGT_NRESET
- net DAP_RX renamed TGT_RX
- net DAP_SWCLK renamed TGT_SWCLK
- net DAP_SWDIO renamed TGT_SWDIO
- net DAP_TX renamed TGT_TX
- net DAP_USB_D+ renamed TGT_USB_D+
- net DAP_USB_D- renamed TGT_USB_D-
Changed lines of the file:
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@@
 </segment>
 </net>
-<net name="DAP_RX" class="0">
+<net name="TGT_RX" class="0">
 <segment>
 <wire x1="170.18" y1="68.58" x2="162.56" y2="68.58" width="0.1524" layer="91"/>
@@
 </segment>
 </net>
-<net name="DAP_USB_D-" class="0">
+<net name="TGT_USB_D-" class="0">
 <segment>
 <wire x1="27.94" y1="96.52" x2="30.48" y2="96.52" width="0.1524" layer="91"/>
@@
 </segment>
 </net>
-<net name="DAP_USB_D+" class="0">
+<net name="TGT_USB_D+" class="0">
 <segment>
 <wire x1="35.56" y1="104.14" x2="27.94" y2="104.14" width="0.1524" layer="91"/>
@@
 </segment>
 </net>
-<net name="DAP_SWCLK" class="0">
+<net name="TGT_SWCLK" class="0">
 <segment>
 <wire x1="162.56" y1="96.52" x2="170.18" y2="96.52" width="0.1524" layer="91"/>
@@
 </segment>
 </net>
-<net name="DAP_SWDIO" class="0">
+<net name="TGT_SWDIO" class="0">
 <segment>
 <wire x1="162.56" y1="93.98" x2="170.18" y2="93.98" width="0.1524" layer="91"/>
@@
 </segment>
 </net>
-<net name="DAP_TX" class="0">
+<net name="TGT_TX" class="0">
 <segment>
 <wire x1="162.56" y1="71.12" x2="170.18" y2="71.12" width="0.1524" layer="91"/>
@@
 </segment>
 </net>
-<net name="DAP_NRESET" class="0">
+<net name="TGT_NRESET" class="0">
 <segment>
 <wire x1="162.56" y1="86.36" x2="170.18" y2="86.36" width="0.1524" layer="91"/>
