File: Bare Design Projects/INTERFACE DAPLink/MK20DX128VFM5/INTERFACE_MK20DX128VFM5.sch (EAGLE design)
At the start: 26 parts, among them CON1 47346-0001, CON2 TC2050-IDC-NL, U2 TLV1117LV33DCYR, U3 IF_MK20DX128VFM5, Y1 CSTCE8M00G55-R0

Commit message: Fixed PDF and name errors
Connections:
- net DAP_NRESET renamed TGT_NRESET
- net DAP_RX renamed TGT_RX
- net DAP_SWCLK renamed TGT_SWCLK
- net DAP_SWDIO renamed TGT_SWDIO
- net DAP_TX renamed TGT_TX
- net DAP_USB_D+ renamed TGT_USB_D+
- net DAP_USB_D- renamed TGT_USB_D-
- net TCLK renamed IF_SWCLK
- net TDI renamed IF_TDI
- net TDO renamed IF_TDO
- net TMS renamed IF_SWDIO
Other:
- note added: "MK20DX128VFM5 DAPLINK Interface"
- note removed: "LCP11u35 DAPLINK Interface"
Changed lines of the file:
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@@
 <sheet>
 <plain>
-<text x="116.84" y="119.38" size="2.54" layer="91">LCP11u35 DAPLINK Interface</text>
+<text x="116.84" y="129.54" size="2.54" layer="91">MK20DX128VFM5 DAPLINK Interface</text>
 <text x="2.54" y="180.34" size="6.4516" layer="90">DAPLINK INTERFACE</text>
 </plain>
@@
 <pinref part="Y1" gate="G$1" pin="3"/>
 <wire x1="106.68" y1="53.34" x2="111.76" y2="53.34" width="0.1524" layer="91"/>
+<junction x="111.76" y="53.34"/>
 </segment>
 </net>
@@
 <pinref part="Y1" gate="G$1" pin="1"/>
 <wire x1="101.6" y1="53.34" x2="96.52" y2="53.34" width="0.1524" layer="91"/>
-</segment>
-</net>
-<net name="DAP_RX" class="0">
+<junction x="96.52" y="53.34"/>
+</segment>
+</net>
+<net name="TGT_RX" class="0">
 <segment>
 <wire x1="170.18" y1="63.5" x2="162.56" y2="63.5" width="0.1524" layer="91"/>
 <label x="170.18" y="63.5" size="2.286" layer="90"/>
 <pinref part="U3" gate="G$1" pin="TGT_RX"/>
-</segment>
-</net>
-<net name="DAP_USB_D-" class="0">
-<segment>
-<wire x1="27.94" y1="96.52" x2="30.48" y2="96.52" width="0.1524" layer="91"/>
-<label x="10.16" y="96.52" size="2.286" layer="90"/>
-<pinref part="R7" gate="G$1" pin="P$1"/>
-</segment>
-<segment>
-<pinref part="CON1" gate="A" pin="D-"/>
-<wire x1="147.32" y1="165.1" x2="152.4" y2="165.1" width="0.1524" layer="91"/>
-<junction x="152.4" y="165.1"/>
-<label x="152.4" y="165.1" size="2.286" layer="90"/>
-</segment>
-</net>
-<net name="DAP_USB_D+" class="0">
-<segment>
-<wire x1="35.56" y1="104.14" x2="27.94" y2="104.14" width="0.1524" layer="91"/>
-<label x="15.24" y="104.14" size="2.286" layer="90"/>
-<pinref part="R4" gate="G$1" pin="P$1"/>
-</segment>
-<segment>
-<pinref part="CON1" gate="A" pin="D+"/>
-<wire x1="147.32" y1="162.56" x2="152.4" y2="162.56" width="0.1524" layer="91"/>
-<junction x="152.4" y="162.56"/>
-<label x="152.4" y="162.56" size="2.286" layer="90"/>
-</segment>
-</net>
-<net name="DAP_SWCLK" class="0">
+<junction x="170.18" y="63.5"/>
+</segment>
+</net>
+<net name="TGT_SWCLK" class="0">
 <segment>
 <wire x1="162.56" y1="91.44" x2="170.18" y2="91.44" width="0.1524" layer="91"/>
 <label x="170.18" y="91.44" size="2.286" layer="90"/>
 <pinref part="U3" gate="G$1" pin="TGT_SWCLK"/>
-</segment>
-</net>
-<net name="DAP_SWDIO" class="0">
+<junction x="170.18" y="91.44"/>
+</segment>
+</net>
+<net name="TGT_SWDIO" class="0">
 <segment>
 <wire x1="162.56" y1="88.9" x2="170.18" y2="88.9" width="0.1524" layer="91"/>
 <label x="170.18" y="88.9" size="2.286" layer="90"/>
 <pinref part="U3" gate="G$1" pin="TGT_SWDIO"/>
-</segment>
-</net>
-<net name="DAP_TX" class="0">
+<junction x="170.18" y="88.9"/>
+</segment>
+</net>
+<net name="TGT_TX" class="0">
 <segment>
 <pinref part="U3" gate="G$1" pin="TGT_TX"/>
 <wire x1="162.56" y1="66.04" x2="170.18" y2="66.04" width="0.1524" layer="91"/>
 <label x="170.18" y="66.04" size="2.286" layer="90"/>
+<junction x="170.18" y="66.04"/>
 </segment>
 </net>
@@
 </segment>
 </net>
-<net name="DAP_NRESET" class="0">
+<net name="TGT_NRESET" class="0">
 <segment>
 <wire x1="81.28" y1="114.3" x2="91.44" y2="114.3" width="0.1524" layer="91"/>
@@
 </segment>
 </net>
-<net name="TMS" class="0">
+<net name="IF_SWDIO" class="0">
 <segment>
 <pinref part="U3" gate="G$1" pin="NC7"/>
@@
 </segment>
 </net>
-<net name="TDO" class="0">
+<net name="IF_TDO" class="0">
 <segment>
 <pinref part="U3" gate="G$1" pin="NC6"/>
@@
 </segment>
 </net>
-<net name="TDI" class="0">
+<net name="IF_TDI" class="0">
 <segment>
 <pinref part="U3" gate="G$1" pin="NC5"/>
@@
 </segment>
 </net>
-<net name="TCLK" class="0">
+<net name="IF_SWCLK" class="0">
 <segment>
 <pinref part="U3" gate="G$1" pin="NC4"/>
@@
 </segment>
 </net>
+<net name="TGT_USB_D+" class="0">
+<segment>
+<wire x1="35.56" y1="104.14" x2="27.94" y2="104.14" width="0.1524" layer="91"/>
+<label x="15.24" y="104.14" size="2.286" layer="90"/>
+<pinref part="R4" gate="G$1" pin="P$1"/>
+<junction x="27.94" y="104.14"/>
+</segment>
+<segment>
+<pinref part="CON1" gate="A" pin="D+"/>
+<wire x1="147.32" y1="162.56" x2="152.4" y2="162.56" width="0.1524" layer="91"/>
+<junction x="152.4" y="162.56"/>
+<label x="152.4" y="162.56" size="2.286" layer="90"/>
+</segment>
+</net>
+<net name="TGT_USB_D-" class="0">
+<segment>
+<wire x1="27.94" y1="96.52" x2="30.48" y2="96.52" width="0.1524" layer="91"/>
+<label x="10.16" y="96.52" size="2.286" layer="90"/>
+<pinref part="R7" gate="G$1" pin="P$1"/>
+<junction x="27.94" y="96.52"/>
+</segment>
+<segment>
+<pinref part="CON1" gate="A" pin="D-"/>
+<wire x1="147.32" y1="165.1" x2="152.4" y2="165.1" width="0.1524" layer="91"/>
+<junction x="152.4" y="165.1"/>
+<label x="152.4" y="165.1" size="2.286" layer="90"/>
+</segment>
+</net>
