File: Bare Design Projects/TARGET/Multitech xDOT/TARGET_xDOT.sch (EAGLE design)
At the start: 11 parts, among them U1 MTXDOT-EU1-A00-1

Commit message: Added LPC11u35 interface macro
Connections:
- net +3.3V_TGT renamed +3.3V
- net NRESET renamed DAP_NRESET
- net SWCLK renamed DAP_SWCLK
- net SWDIO renamed DAP_SWDIO
- net UART0_RX renamed DAP_RX
- net UART0_TX renamed DAP_TX
Changed lines of the file:
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@@
 <part name="C1" library="mbed-HDK-RLCQ" deviceset="CAPACITOR" device="0603" value="10uF"/>
 <part name="GND8" library="mbed-HDK-misc-Symbol" deviceset="GND" device=""/>
-<part name="PWR1" library="mbed-HDK-misc-Symbol" deviceset="+3.3V_TGT" device=""/>
 <part name="C2" library="mbed-HDK-RLCQ" deviceset="CAPACITOR" device="0603" value="100nF"/>
 <part name="GND9" library="mbed-HDK-misc-Symbol" deviceset="GND" device=""/>
@@
 <part name="C7" library="mbed-HDK-RLCQ" deviceset="CAPACITOR" device="0402" value="6.8pF"/>
 <part name="GND13" library="mbed-HDK-misc-Symbol" deviceset="GND" device=""/>
+<part name="PWR1" library="mbed-HDK-misc-Symbol" deviceset="+3.3V" device=""/>
 </parts>
 <sheets>
@@
 </instance>
 <instance part="GND8" gate="1" x="-10.16" y="83.82" rot="R90"/>
-<instance part="PWR1" gate="G$1" x="-33.02" y="86.36"/>
 <instance part="C2" gate="G$1" x="-17.78" y="78.74" smashed="yes" rot="R90">
 <attribute name="NAME" x="-13.462" y="80.264" size="1.27" layer="95" font="vector" ratio="12" rot="R180"/>
@@
 </instance>
 <instance part="GND13" gate="1" x="116.84" y="30.48" rot="R90"/>
+<instance part="PWR1" gate="G$1" x="-33.02" y="86.36"/>
 </instances>
 <busses>
@@
 </segment>
 </net>
-<net name="UART0_TX" class="0">
+<net name="DAP_TX" class="0">
 <segment>
 <pinref part="U1" gate="G$1" pin="UART0_TX"/>
@@
 </segment>
 </net>
-<net name="UART0_RX" class="0">
+<net name="DAP_RX" class="0">
 <segment>
 <pinref part="U1" gate="G$1" pin="UART0_RX"/>
@@
 </segment>
 </net>
-<net name="SWCLK" class="0">
+<net name="DAP_SWCLK" class="0">
 <segment>
 <pinref part="U1" gate="G$1" pin="SWCLK"/>
@@
 </segment>
 </net>
-<net name="SWDIO" class="0">
+<net name="DAP_SWDIO" class="0">
 <segment>
 <pinref part="U1" gate="G$1" pin="SWDIO"/>
 <wire x1="38.1" y1="73.66" x2="78.74" y2="73.66" width="0.1524" layer="91"/>
 <junction x="78.74" y="73.66"/>
-<label x="70.612" y="73.66" size="1.778" layer="95"/>
+<label x="65.532" y="73.66" size="1.778" layer="95"/>
 </segment>
 </net>
@@
 </segment>
 </net>
-<net name="NRESET" class="0">
+<net name="DAP_NRESET" class="0">
 <segment>
 <pinref part="U1" gate="G$1" pin="NRESET"/>
 <wire x1="38.1" y1="66.04" x2="78.74" y2="66.04" width="0.1524" layer="91"/>
 <junction x="78.74" y="66.04"/>
-<label x="69.342" y="66.04" size="1.778" layer="95"/>
+<label x="64.262" y="66.04" size="1.778" layer="95"/>
 </segment>
 </net>
@@
 <junction x="78.74" y="30.48"/>
 <label x="72.39" y="30.48" size="1.778" layer="95"/>
-</segment>
-</net>
-<net name="+3.3V_TGT" class="0">
-<segment>
-<pinref part="U1" gate="G$1" pin="VDD(1)"/>
-<wire x1="-5.08" y1="66.04" x2="-33.02" y2="66.04" width="0.1524" layer="91"/>
-<wire x1="-33.02" y1="66.04" x2="-33.02" y2="68.58" width="0.1524" layer="91"/>
-<pinref part="U1" gate="G$1" pin="VDD(0)"/>
-<wire x1="-33.02" y1="68.58" x2="-5.08" y2="68.58" width="0.1524" layer="91"/>
-<junction x="-33.02" y="68.58"/>
-<wire x1="-33.02" y1="68.58" x2="-33.02" y2="78.74" width="0.1524" layer="91"/>
-<pinref part="C1" gate="G$1" pin="P$1"/>
-<wire x1="-33.02" y1="78.74" x2="-33.02" y2="83.82" width="0.1524" layer="91"/>
-<wire x1="-33.02" y1="83.82" x2="-20.32" y2="83.82" width="0.1524" layer="91"/>
-<junction x="-33.02" y="83.82"/>
-<pinref part="PWR1" gate="G$1" pin="+3.3V_TGT"/>
-<wire x1="-33.02" y1="83.82" x2="-33.02" y2="86.36" width="0.1524" layer="91"/>
-<wire x1="-33.02" y1="78.74" x2="-20.32" y2="78.74" width="0.1524" layer="91"/>
-<pinref part="C2" gate="G$1" pin="P$1"/>
-<junction x="-33.02" y="78.74"/>
 </segment>
 </net>
@@
 </segment>
 </net>
+<net name="+3.3V" class="0">
+<segment>
+<pinref part="U1" gate="G$1" pin="VDD(1)"/>
+<wire x1="-5.08" y1="66.04" x2="-33.02" y2="66.04" width="0.1524" layer="91"/>
+<wire x1="-33.02" y1="66.04" x2="-33.02" y2="68.58" width="0.1524" layer="91"/>
+<pinref part="U1" gate="G$1" pin="VDD(0)"/>
+<wire x1="-33.02" y1="68.58" x2="-5.08" y2="68.58" width="0.1524" layer="91"/>
+<junction x="-33.02" y="68.58"/>
+<wire x1="-33.02" y1="68.58" x2="-33.02" y2="78.74" width="0.1524" layer="91"/>
+<pinref part="C1" gate="G$1" pin="P$1"/>
+<wire x1="-33.02" y1="78.74" x2="-33.02" y2="83.82" width="0.1524" layer="91"/>
+<wire x1="-33.02" y1="83.82" x2="-20.32" y2="83.82" width="0.1524" layer="91"/>
+<junction x="-33.02" y="83.82"/>
+<wire x1="-33.02" y1="83.82" x2="-33.02" y2="86.36" width="0.1524" layer="91"/>
+<wire x1="-33.02" y1="78.74" x2="-20.32" y2="78.74" width="0.1524" layer="91"/>
+<pinref part="C2" gate="G$1" pin="P$1"/>
+<junction x="-33.02" y="78.74"/>
+<pinref part="PWR1" gate="G$1" pin="+3.3V"/>
+</segment>
+</net>

Commit message: Updated design removed obsolete components
Parts:
- removed C5: 10pF, mbed-HDK-RLCQ:CAPACITOR0402
- removed L1: 7.5uH, mbed-HDK-RLCQ:INDUCTOR0402
- removed R1: 0, mbed-HDK-RLCQ:RESISTOR0402
- C3: value 6.8pF -> 9.1pF
- C4: value 10pF -> 5.6pF
Connections:
- net DAP_NRESET renamed TGT_NRESET
- net DAP_SWCLK renamed TGT_SWCLK
- net DAP_SWDIO renamed TGT_SWDIO
- net UART1_RX renamed TGT_RX
- net UART1_TX renamed TGT_TX
- net ANT1: no longer L1.P$1, R1.P$1
- net GND: no longer C5.P$1
- net N$4: no longer C5.P$2, L1.P$2, R1.P$2
Other:
- note added: ""C3" Default = 9.1pF (800MHz) Default = 6.8pF (900MHz)"
- note added: ""C4" Default = 5.6pF (800MHz) Default = 7.5pF (900MHz)"
- note added: "TARGET"
- moved on the sheet: ANT1, C1, C2, C3, C4, C6, C7, U1
